Commit message: added_gazebo

File: description/robot.urdf.xacro (robot description, xacro)
@@ -14,4 +14,5 @@
     </material>
     <xacro:include filename="robot_core.xacro" />
+    <xacro:include filename="gazebo_control.xacro"/>
     <xacro:include filename="lidar.xacro" />
 </robot>

File: description/robot_core.xacro (robot description, xacro)
@@ -29,4 +29,7 @@
         </xacro:inertial_box>
     </link>
+    <gazebo reference="chassis">
+        <material>Gazebo/White</material>
+    </gazebo>
 <!-- LEFT WHEEL LINK -->
     <joint name="left_wheel_joint" type="continuous">
@@ -34,5 +37,5 @@
         <child link ="left_wheel"/>
         <origin xyz="0 0.125 0" rpy="${pi/2} 0 0"/>
-        <axis xyz="0 0 1"/>
+        <axis xyz="0 0 -1"/>
     </joint>
     <link name='left_wheel'>
@@ -52,4 +55,7 @@
         </xacro:inertial_cylinder>
     </link>
+    <gazebo reference="left_wheel">
+        <material>Gazebo/Blue</material>
+    </gazebo>
 <!-- RIGHT WHEEL LINK -->
     <joint name="right_wheel_joint" type="continuous">
@@ -57,5 +63,5 @@
         <child link ="right_wheel"/>
         <origin xyz="0 -0.125 0" rpy="-${pi/2} 0 0"/>
-        <axis xyz="0 0 -1"/>
+        <axis xyz="0 0 1"/>
     </joint>
     <link name='right_wheel'>
@@ -75,4 +81,7 @@
         </xacro:inertial_cylinder>
     </link>
+    <gazebo reference="right_wheel">
+        <material>Gazebo/Blue</material>
+    </gazebo>
 <!-- LEFT CASTER WHEEL LINK -->
     <joint name="left_caster_wheel_link" type="fixed">
@@ -97,4 +106,9 @@
         </xacro:inertial_sphere>
     </link>
+    <gazebo reference="left_caster_wheel">
+        <material>Gazebo/Orange</material>
+        <mu1 value="0.001"/>
+        <mu2 value="0.001"/>
+    </gazebo>
 <!-- RIGHT CASTER WHEEL LINK -->
     <joint name="right_caster_wheel_link" type="fixed">
@@ -119,3 +133,8 @@
         </xacro:inertial_sphere>
     </link>
+    <gazebo reference="right_caster_wheel">
+        <material>Gazebo/Orange</material>
+        <mu1 value="0.001"/>
+        <mu2 value="0.001"/>
+    </gazebo>
 </robot>
