Commit message: slam working

File: description/robot_core.xacro (robot description, xacro)
@@ -4,4 +4,12 @@
 <!-- BASE LINK -->
     <link name='base_link'>
+    </link>
+<!-- BASE FOOTPRINT LINK -->
+    <joint name="base_footprint_joint" type="fixed">
+        <parent link="base_link"/>
+        <child link ="base_footprint"/>
+        <origin xyz="0 0 0" ryp="0 0 0"/>
+    </joint>
+    <link name='base_footprint'>
     </link>
 <!-- CHASSIS LINK -->
